File: Connectors.kicad_sch (KiCad schematic)
At the start: 0 parts

Commit message: Improvements
Switched ADC to ADC128S.
Upgraded USB to USB-C
Improved Analog front end to work with signals better.
Parts:
- added J402: SWD, Connector_PinHeader_2.54mm:PinHeader_2x03_P2.54mm_Vertical, symbol Connector_Generic:Conn_02x03_Odd_Even
- added J501: GPIO, Connector_PinHeader_2.54mm:PinHeader_1x07_P2.54mm_Vertical, symbol Connector_Generic:Conn_01x07
- added J502: VCC, Connector_PinHeader_2.54mm:PinHeader_1x07_P2.54mm_Vertical, symbol Connector_Generic:Conn_01x07
- added J503: GND, Connector_PinHeader_2.54mm:PinHeader_1x07_P2.54mm_Vertical, symbol Connector_Generic:Conn_01x07
Connections:
- new net +3.3V: J402.1 (Pin_1), J502.1 (Pin_1), J502.2 (Pin_2), J502.3 (Pin_3), J502.4 (Pin_4), J502.5 (Pin_5), J502.6 (Pin_6), J502.7 (Pin_7)
- new net GND: J402.3 (Pin_3), J402.5 (Pin_5), J503.1 (Pin_1), J503.2 (Pin_2), J503.3 (Pin_3), J503.4 (Pin_4), J503.5 (Pin_5), J503.6 (Pin_6), J503.7 (Pin_7)
- new net MCU_GPIO_PB00: J501.5 (Pin_5)
- new net MCU_GPIO_PB01: J501.4 (Pin_4)
- new net MCU_GPIO_PB02: J501.3 (Pin_3)
- new net MCU_GPIO_PB10: J501.2 (Pin_2)
- new net MCU_GPIO_PB11: J501.1 (Pin_1)
- new net MCU_GPIO_PC04: J501.7 (Pin_7)
- new net MCU_GPIO_PC05: J501.6 (Pin_6)
- new net MCU_NRST: J402.6 (Pin_6)
- new net MCU_SWD_CLK: J402.4 (Pin_4)
- new net MCU_SWD_IO: J402.2 (Pin_2)
Other:
- note added: "GPIO"
- note added: "SWD"
